Commit message: more accurate model

File: MOMA_project/src/amr_visualisation/urdf/LD250.urdf (robot description, URDF)
Before this commit: robot LD90, 2 links, 1 joints
Links:
- link main_body: geometry collision mesh filename=package://amr_visualisation/meshes/amr_chassis_scaled.stl; visual mesh filename=package://amr_visualisation/meshes/amr_chassis_scaled.stl
