Commit message: moveit redefined for moma

File: MOMA_project/src/amr_visualisation/urdf/amr_core.xacro (robot description, xacro)
@@ -39,3 +39,159 @@
     <origin xyz="0 0 0.15"/>
   </joint>
+<link name="left_wheel">
+    <visual>
+      <origin rpy="1.5707963267949 0 0" xyz="0 0 0"/>
+      <geometry>
+        <cylinder length="0.03937" radius="0.088"/>
+      </geometry>
+      <material name="amr_wheel_color"/>
+    </visual>
+    <collision>
+      <origin rpy="1.5707963267949 0 0" xyz="0 0 0"/>
+      <geometry>
+        <cylinder length="0.03937" radius="0.088"/>
+      </geometry>
+    </collision>
+    <inertial>
+      <mass value="0.17"/>
+      <inertia ixx="0.000204" ixy="0.0" ixz="0.0" iyy="0.000306" iyz="0.0" izz="0.000204"/>
+    </inertial>
+  </link>
+  <joint name="left_wheel_joint" type="continuous">
+    <axis rpy="0 0 0" xyz="0 1 0"/>
+    <parent link="amr_main_body"/>
+    <child link="left_wheel"/>
+    <!-- <origin rpy="0 0 0" xyz="0 0.3 0.000881"/> -->
+    <origin rpy="0 0 0" xyz="-0.004 0.3025 0.000881"/>
+  </joint>
+  <link name="right_wheel">
+    <visual>
+      <origin rpy="1.5707963267949 0 0" xyz="0 0 0"/>
+      <geometry>
+        <cylinder length="0.03937" radius="0.088"/>
+      </geometry>
+      <material name="amr_wheel_color"/>
+    </visual>
+    <collision>
+      <origin rpy="1.5707963267949 0 0" xyz="0 0 0"/>
+      <geometry>
+        <cylinder length="0.03937" radius="0.088"/>
+      </geometry>
+    </collision>
+    <inertial>
+      <mass value="0.17"/>
+      <inertia ixx="0.000204" ixy="0.0" ixz="0.0" iyy="0.000306" iyz="0.0" izz="0.000204"/>
+    </inertial>
+  </link>
+  <joint name="right_wheel_joint" type="continuous">
+    <axis rpy="0 0 0" xyz="0 1 0"/>
+    <parent link="amr_main_body"/>
+    <child link="right_wheel"/>
+    <!-- <origin rpy="0 0 0" xyz="0 -0.3 0.000881"/> -->
+    <origin rpy="0 0 0" xyz="-0.004 -0.3025 0.000881"/>
+  </joint>
+  <link name="right_front_small_wheel">
+    <visual>
+      <origin rpy="1.5707963267949 0 0" xyz="0 0 0"/>
+      <geometry>
+        <cylinder length="0.02775" radius="0.03625"/>
+      </geometry>
+      <material name="amr_wheel_color"/>
+    </visual>
+    <collision>
+      <origin rpy="1.5707963267949 0 0" xyz="0 0 0"/>
+      <geometry>
+        <cylinder length="0.02775" radius="0.03625"/>
+      </geometry>
+    </collision>
+    <inertial>
+      <mass value="0.17"/>
+      <inertia ixx="0.000204" ixy="0.0" ixz="0.0" iyy="0.000306" iyz="0.0" izz="0.000204"/>
+    </inertial>
+  </link>
+  <joint name="right_front_small_wheel_joint" type="continuous">
+    <axis rpy="0 0 0" xyz="0 1 0"/>
+    <parent link="amr_main_body"/>
+    <child link="right_front_small_wheel"/>
+    <!-- <origin rpy="0 0 0" xyz="0.209 -0.108 -0.049"/> -->
+    <origin rpy="0 0 0" xyz="0.2493 -0.2325 -0.049"/>
+  </joint>
+  <link name="left_front_small_wheel">
+    <visual>
+      <origin rpy="1.5707963267949 0 0" xyz="0 0 0"/>
+      <geometry>
+        <cylinder length="0.02775" radius="0.03625"/>
+      </geometry>
+      <material name="amr_wheel_color"/>
+    </visual>
+    <collision>
+      <origin rpy="1.5707963267949 0 0" xyz="0 0 0"/>
+      <geometry>
+        <cylinder length="0.02775" radius="0.03625"/>
+      </geometry>
+    </collision>
+    <inertial>
+      <mass value="0.17"/>
+      <inertia ixx="0.000204" ixy="0.0" ixz="0.0" iyy="0.000306" iyz="0.0" izz="0.000204"/>
+    </inertial>
+  </link>
+  <joint name="left_front_small_wheel_joint" type="continuous">
+    <axis rpy="0 0 0" xyz="0 1 0"/>
+    <parent link="amr_main_body"/>
+    <child link="left_front_small_wheel"/>
+    <!-- <origin rpy="0 0 0" xyz="0.209 0.108 -0.049"/> -->
+    <origin rpy="0 0 0" xyz="0.2493 0.2325 -0.049"/>
+  </joint>
+  <link name="left_back_small_wheel">
+    <visual>
+      <origin rpy="1.5707963267949 0 0" xyz="0 0 0"/>
+      <geometry>
+        <cylinder length="0.02775" radius="0.03625"/>
+      </geometry>
+      <material name="amr_wheel_color"/>
+    </visual>
+    <collision>
+      <origin rpy="1.5707963267949 0 0" xyz="0 0 0"/>
+      <geometry>
+        <cylinder length="0.02775" radius="0.03625"/>
+      </geometry>
+    </collision>
+    <inertial>
+      <mass value="0.17"/>
+      <inertia ixx="0.000204" ixy="0.0" ixz="0.0" iyy="0.000306" iyz="0.0" izz="0.000204"/>
+    </inertial>
+  </link>
+  <joint name="left_back_small_wheel_joint" type="continuous">
+    <axis rpy="0 0 0" xyz="0 1 0"/>
+    <parent link="amr_main_body"/>
+    <child link="left_back_small_wheel"/>
+    <!-- <origin rpy="0 0 0" xyz="-0.228 0.156 -0.049"/> -->
+    <origin rpy="0 0 0" xyz="-0.257 0.2325 -0.049"/>
+  </joint>
+  <link name="right_back_small_wheel">
+    <visual>
+      <origin rpy="1.5707963267949 0 0" xyz="0 0 0"/>
+      <geometry>
+        <cylinder length="0.02775" radius="0.03625"/>
+      </geometry>
+      <material name="amr_wheel_color"/>
+    </visual>
+    <collision>
+      <origin rpy="1.5707963267949 0 0" xyz="0 0 0"/>
+      <geometry>
+        <cylinder length="0.02775" radius="0.03625"/>
+      </geometry>
+    </collision>
+    <inertial>
+      <mass value="0.17"/>
+      <inertia ixx="0.000204" ixy="0.0" ixz="0.0" iyy="0.000306" iyz="0.0" izz="0.000204"/>
+    </inertial>
+  </link>
+  <joint name="right_back_small_wheel_joint" type="continuous">
+    <axis rpy="0 0 0" xyz="0 1 0"/>
+    <parent link="amr_main_body"/>
+    <child link="right_back_small_wheel"/>
+    <!-- <origin rpy="0 0 0" xyz="-0.228 -0.156 -0.049"/> -->
+    <origin rpy="0 0 0" xyz="-0.257 -0.2325 -0.049"/>
+  </joint>
 </robot>

File: MOMA_project/src/amr_visualisation/urdf/tm12s_core.xacro (robot description, xacro)
@@ -11,7 +11,7 @@
   <!-- you must modify 'macro.tm12s-nominal.urdf.xacro' to 'user_defined.urdf.xacro'  -->
   <xacro:include filename="macro.tm12s-nominal.urdf.xacro" />
-  <xacro:include filename="macro.gazebo.xacro" />
+  <!-- <xacro:include filename="macro.gazebo.xacro" /> -->
   <!--  -->
-  <xacro:tmr_gazebo ns="$(arg ns)" prefix="$(arg prefix)" />
+  <!-- <xacro:tmr_gazebo ns="$(arg ns)" prefix="$(arg prefix)" /> -->
   <xacro:tmr_transmission prefix="$(arg prefix)" hw_iface="$(arg trans_hw_iface)" />
   <xacro:tmr_materials/>
